File: ESProg_ESP8266_Template_Horizontal.kicad_pcb (KiCad board)
At the start: 2 copper layers, 55.3 x 32 mm, 10 parts, among them P1 ESProg Mating Header, SW1 RESET, U1 ESP-12E

Commit message: Some improvements
Vertical footprint added
Other:
- board text added: "Programming demo with ESProg"
- board text removed: "Programming with ESProg"
Changed lines of the file:
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@@
   (gr_arc (start 108 104) (end 105 104) (angle -90) (layer Edge.Cuts) (width 0.15))
   (gr_arc (start 108 78) (end 108 75) (angle -90) (layer Edge.Cuts) (width 0.15))
-  (gr_text "Programming with\nESProg" (at 154 104) (layer F.SilkS)
+  (gr_text "Programming demo\nwith ESProg" (at 154 104) (layer F.SilkS)
     (effects (font (size 1.2 1.2) (thickness 0.25)) (justify right))
   )
